Commit message: Updated this alternate glennan_2nd_flr package to work with the turtlebot simulation.
The remaining remnants in this forked version from the cwru_robotics repository had all the remaining package dependencies removed.

File: glennan_2nd_flr.urdf (robot description, URDF)
Before this commit: robot glennan_2nd_floor, 2 links, 1 joints
Links:
- removed link link
- added link glennan_map, mass 1000; collision mesh filename=package://glennan_second_floor/glennan_2nd_flr.stl; visual mesh filename=package://glennan_second_floor/glennan_2nd_flr.stl
Joints:
- joint glue_robot_to_world: child link -> glennan_map
